File: KiCad/NR24_Schematic/Ti_Board.kicad_sch (KiCad schematic)
At the start: 8 parts, among them J5 Dash TI Connection, J5 J1 Pin J3 Pin, J5 J12 (CAN Interface w/ Transce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, J5 J4 Pin J2 Pin, J5 J5 Pin J7 Pin, J5 J8 Pin J6 Pin, J6 SpeakON_NL2, J8 CAN Connector

Commit message: New Ti Board
Parts:
- added D2, D3: 1N5402, Diode_THT:D_DO-201AD_P15.24mm_Horizontal, symbol Diode:1N5402
- added J5: XBEE PRO, symbol Connector_Generic:Conn_02x06_Counter_Clockwise
- added Q1, Q2, Q3: Q_NMOS_DGS, symbol Device:Q_NMOS_DGS
- added R1, R2, R3, R4: 10K Ω 5%, symbol Device:R_US
Connections:
- net BLK: now reaches J5.60 (GND)
- net Yellow (3.3 Xbee): now reaches J5.41 (3.3V)
- net Blue (Xbee): now reaches J5.43 (GPIO139)
- net Purple (Xbee): now reaches J5.44 (GPIO56)
- new net: Q1.1 (D), R3.2
- new net: Q1.3 (S), Q2.2 (G), R3.1, R4.1
- new net: Q2.1 (D), R4.2
- new net: D3.1 (K), R2.1
- new net: D2.1 (K), R1.1
- new net Blue: J5.4 (TX)
- new net Grey -> Black: J5.2 (GND)
- new net High Input: R2.2
- new net Purple: J5.3 (RX)
- new net White -> Yellow: J5.1 (3.3V)
- new net in_BLK: D3.2 (A), Q1.2 (G)
Other:
- moved on the sheet: J5, J8
