File: KiCad/NR24_Schematic/AMS.kicad_sch (KiCad schematic)
At the start: 0 parts

Commit message: Now it works :)
Parts:
- added BT1, BT2: Battery, symbol Device:Battery
- added U? (x2): Orion_Jr._2_BMS, symbol CamachosSymbols:Sevcon_Gen4_Size6
Connections:
- new net: BT1.1 (+), BT2.2 (-)
- new net AIR: U?.15 (Multi_Purpose_Input), U?.15 (Multi_Purpose_Input)
- new net CAN_GND: U?.6 (Ground), U?.6 (Ground)
- new net CAN_High: U?.20 (CAN_high), U?.20 (CAN_high)
- new net CAN_Low: U?.19 (CAN_low), U?.19 (CAN_low)
- new net Charge Sig: U?.5 (Charger_Safety), U?.5 (Charger_Safety)
- new net HV +: BT2.1 (+)
- new net HV -: BT1.2 (-)
- new net TI Board: U?.2 (Ready_Power), U?.2 (Ready_Power), U?.4 (Charge_Power), U?.4 (Charge_Power)

Commit message: uh
Connections:
- net TI Board renamed LV_sys (for charging)
- net LV_sys (for charging): no longer U?.2 (Ready_Power), U?.2 (Ready_Power)
- new net LV_sys (for discharge): U?.2 (Ready_Power), U?.2 (Ready_Power)
Other:
- note added: "CAN Bus"
- moved on the sheet: BT1, BT2

Commit message: Updates
Connections:
- net LV_sys (for charging) renamed LV_pwr (chrg)
- net LV_sys (for discharge) renamed LV_pwr (dchrg)
Changed lines of the file:
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@@
 (kicad_sch (version 20230121) (generator eeschema)
   (paper "A4")
-  (junction (at 181.61 154.94) (diameter 0) (color 0 0 0 0)
+  (junction (at 154.94 154.94) (diameter 0) (color 0 0 0 0)
   )
   (bus_entry (at 152.4 55.88) (size 2.54 2.54)
@@
     (stroke (width 0.75) (type default) (color 0 132 132 1))
   )
-  (wire (pts (xy 181.61 154.94) (xy 251.46 154.94))
+  (wire (pts (xy 154.94 154.94) (xy 251.46 154.94))
     (stroke (width 0) (type default))
   )
@@
     (stroke (width 0) (type default))
   )
-  (wire (pts (xy 59.69 154.94) (xy 181.61 154.94))
+  (wire (pts (xy 59.69 154.94) (xy 154.94 154.94))
     (stroke (width 0) (type default))
   )
@@
     (stroke (width 1) (type default))
   )
-  (wire (pts (xy 181.61 154.94) (xy 181.61 158.75))
+  (wire (pts (xy 154.94 154.94) (xy 154.94 158.75))
     (stroke (width 0) (type default))
   )
@@
   )
   (text_box "Different wiring harnesses for charging vs driving? While driving will we need Charge Power pin in order to implement regenerative braking?"
-    (at 129.54 138.43 0) (size 39.37 11.43)
+    (at 137.16 132.08 0) (size 39.37 11.43)
     (stroke (width 0.5) (type default) (color 255 0 0 1))
     (fill (type none))
@@
     (effects (font (size 1.5 1.5) (color 0 72 72 1)) (justify left bottom))
   )
-  (hierarchical_label "LV_sys (for charging)" (shape input) (at 146.05 113.03 270) (fields_autoplaced)
+  (hierarchical_label "LV_pwr (chrg)" (shape input) (at 146.05 113.03 270) (fields_autoplaced)
     (effects (font (size 1.27 1.27) (thickness 0.254) bold (color 255 0 0 1)) (justify right))
   )
@@
     (effects (font (size 1.27 1.27)) (justify right))
   )
-  (hierarchical_label "LV_sys (for discharge)" (shape input) (at 161.29 113.03 270) (fields_autoplaced)
+  (hierarchical_label "LV_pwr (dchrg)" (shape input) (at 161.29 113.03 270) (fields_autoplaced)
     (effects (font (size 1.27 1.27) (thickness 0.254) bold (color 255 0 0 1)) (justify right))
   )
@@
     (effects (font (size 1.27 1.27)) (justify left))
   )
-  (hierarchical_label "LV_sys (for discharge)" (shape input) (at 151.13 111.76 270) (fields_autoplaced)
+  (hierarchical_label "LV_pwr (dchrg)" (shape input) (at 151.13 111.76 270) (fields_autoplaced)
     (effects (font (size 1.27 1.27) (thickness 0.254) bold (color 255 0 0 1)) (justify right))
   )
@@
     (effects (font (size 1.27 1.27)) (justify left))
   )
-  (hierarchical_label "AIR" (shape input) (at 181.61 158.75 270) (fields_autoplaced)
+  (hierarchical_label "AIR" (shape input) (at 154.94 158.75 270) (fields_autoplaced)
     (effects (font (size 1.27 1.27)) (justify right))
   )
@@
     (effects (font (size 1.27 1.27)) (justify left))
   )
-  (hierarchical_label "LV_sys (for charging)" (shape input) (at 166.37 113.03 270) (fields_autoplaced)
-    (effects (font (size 1.27 1.27) (thickness 0.254) bold (color 255 0 0 1)) (justify right))
-  )
+  (hierarchical_label "LV_pwr (chrg)" (shape input) (at 166.37 113.03 270) (fields_autoplaced)
+    (effects (font (size 1.27 1.27) (thickness 0.254) bold (color 255 0 0 1)) (justify right))
+  )

Commit message: Root Update
Connections:
- net HV + renamed HV + High A
Changed lines of the file:
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@@
   (junction (at 154.94 154.94) (diameter 0) (color 0 0 0 0)
   )
+  (junction (at 135.89 179.07) (diameter 0) (color 0 0 0 0)
+  )
   (bus_entry (at 152.4 55.88) (size 2.54 2.54)
     (stroke (width 0) (type default))
@@
     (stroke (width 0.75) (type default) (color 0 132 132 1))
   )
+  (wire (pts (xy 135.89 168.91) (xy 143.51 168.91))
+    (stroke (width 1) (type default))
+  )
   (wire (pts (xy 166.37 92.71) (xy 166.37 113.03))
     (stroke (width 0) (type default) (color 132 0 0 1))
@@
     (stroke (width 0) (type default))
   )
+  (wire (pts (xy 135.89 179.07) (xy 135.89 168.91))
+    (stroke (width 1) (type default))
+  )
   (wire (pts (xy 181.61 85.09) (xy 161.29 85.09))
     (stroke (width 0) (type default) (color 132 0 0 1))
@@
     (stroke (width 0) (type default))
   )
+  (wire (pts (xy 135.89 179.07) (xy 143.51 179.07))
+    (stroke (width 1) (type default))
+  )
   (wire (pts (xy 181.61 92.71) (xy 166.37 92.71))
     (stroke (width 0) (type default) (color 132 0 0 1))
@@
     (stroke (width 0) (type default) (color 132 0 0 1))
   )
-  (wire (pts (xy 143.51 179.07) (xy 130.81 179.07))
+  (wire (pts (xy 130.81 179.07) (xy 135.89 179.07))
     (stroke (width 1) (type default))
   )
@@
     (effects (font (size 1.27 1.27)) (justify left))
   )
-  (hierarchical_label "HV +" (shape input) (at 143.51 179.07 0) (fields_autoplaced)
+  (hierarchical_label "HV + High A" (shape input) (at 143.51 179.07 0) (fields_autoplaced)
     (effects (font (size 1.27 1.27)) (justify left))
   )
@@
     (effects (font (size 1.27 1.27)) (justify left))
   )
+  (hierarchical_label "HV + Low A" (shape input) (at 143.51 168.91 0) (fields_autoplaced)
+    (effects (font (size 1.27 1.27)) (justify left))
+  )

Commit message: NOV1 Changes w Clarks
Parts:
- added D1: 1N4001, Diode_THT:D_DO-41_SOD81_P10.16mm_Horizontal, symbol Diode:1N4001
- added SW?: AMS Fault Reset Button, symbol CamachosSymbols:Safety Switch
- added U?: LY3 DC12 (Relay), symbol CamachosSymbols:Sevcon_Gen4_Size6
Connections:
- net AMS Fault: now reaches U?.9 (Multi_Purpose_Output_1)
- net AMS Fault: now also U?.9 (Multi_Purpose_Output_1), SW?.1 (A), U?.3 (SPDT3)
- net AIR renamed STDWN_CT_OUT
- net STDWN_CT_OUT: now also U?.8 (TermB2)
- new net: D1.1 (K), SW?.2 (B), U?.11 (High_IN), U?.9 (TermB3)
- new net Dash_Error +: U?.4 (TermA1)
- new net Dash_Error -: U?.1 (STDP1)
- new net GND: D1.2 (A), U?.12 (Low_IN)
- new net STDWN_CT_IN: U?.2 (SPDT2)

Commit message: ams with IMD inside
Parts:
- removed U?: Orion_Jr._2_BMS, symbol CamachosSymbols:Sevcon_Gen4_Size6
- added D1: 1N4001, Diode_THT:D_DO-41_SOD81_P10.16mm_Horizontal, symbol Diode:1N4001
- added SW?: IMD Fault Reset Button, symbol CamachosSymbols:Safety Switch
- added U?: ISOMETER_IR155-3203, symbol CamachosSymbols:Sevcon_Gen4_Size6
- added U?: LY3 DC12 (Relay), symbol CamachosSymbols:Sevcon_Gen4_Size6
- added U?: Orion_Jr._2_BMS, symbol CamachosSymbols:Sevcon_Gen4_Size6
Connections:
- net LV_pwr (dchrg) is gone; now on net LV_pwr: U?.2 (Ready_Power)
- net AMS Fault: now also U?.9 (Multi_Purpose_Output_1)
- net Charge Sig: now also U?.5 (Charger_Safety)
- net Dash_Error +: now also U?.4 (TermA1)
- net Dash_Error -: now also U?.1 (STDP1)
- net GND: now also D1.2 (A), U?.1 (Line_Voltage(XLA+)), U?.12 (Low_IN), U?.3 (Chassis_Ground), U?.4 (Chassis_Ground)
- net HV + High A: now also U?.1 (Line_Voltage(XLA+)), U?.2 (Supply_Voltage)
- net CAN_GND renamed CAN_Ground
- net LV_pwr (chrg) renamed LV_pwr
- net LV_pwr: now also U?.2 (Ready_Power), U?.4 (Charge_Power)
- net STDWN_CT_IN: no longer names the net of U?.2 (SPDT2)
- net STDWN_CT_IN: now also U?.2 (SPDT2)
- net STDWN_CT_OUT renamed STDWN_CT_IN1
- net STDWN_CT_IN1: no longer U?.15 (Multi_Purpose_Input)
- new net: SW?.1 (A), U?.3 (SPDT3), U?.8 (Status_Output(high_side))
- new net: D1.1 (K), SW?.2 (B), U?.11 (High_IN), U?.9 (TermB3)
- new net LV_High: U?.2 (Supply_Voltage)
- new net STDWN_CT_OUT1: U?.15 (Multi_Purpose_Input), U?.15 (Multi_Purpose_Input)
- new net STDWN_CT_OUT2: U?.8 (TermB2)
Other:
- moved on the sheet: BT1, BT2, D1

Commit message: hm
Parts:
- U? (x2): value LY3 DC12 (Relay) -> Grainger Relay
Changed lines of the file:
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@@
       (effects (font (size 2 2)) hide)
     )
-    (property "Value" "LY3 DC12 (Relay)" (at 252.73 151.13 0)
+    (property "Value" "Grainger Relay" (at 252.73 151.13 0)
       (effects (font (size 1.27 1.27)) (justify right top))
     )
@@
       (effects (font (size 2 2)) hide)
     )
-    (property "Value" "LY3 DC12 (Relay)" (at 246.38 85.09 0)
+    (property "Value" "Grainger Relay" (at 246.38 85.09 0)
       (effects (font (size 1.27 1.27)) (justify right top))
     )
