File: KiCad/NR24_Schematic/AMS.kicad_sch (KiCad schematic)
At the start: 9 parts

Commit message: Small Stuff update
Connections:
- net HV -: now also U?.2 (Supply_Voltage)
Other:
- note added: "7 AMP fuse installed by power train"
Changed lines of the file:
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@@
   (junction (at 210.82 149.86) (diameter 0) (color 0 0 0 0)
   )
+  (junction (at 82.55 48.26) (diameter 0) (color 0 0 0 0)
+  )
   (junction (at 105.41 146.05) (diameter 0) (color 0 0 0 0)
   )
@@
   )
   (wire (pts (xy 91.44 31.75) (xy 121.92 31.75))
+    (stroke (width 1) (type default))
+  )
+  (wire (pts (xy 116.84 52.07) (xy 82.55 52.07))
     (stroke (width 1) (type default))
   )
@@
     (stroke (width 0) (type default))
   )
+  (wire (pts (xy 116.84 52.07) (xy 116.84 91.44))
+    (stroke (width 1) (type default))
+  )
   (wire (pts (xy 245.11 40.64) (xy 251.46 40.64))
     (stroke (width 0) (type default))
@@
     (stroke (width 0) (type default))
   )
+  (wire (pts (xy 82.55 52.07) (xy 82.55 48.26))
+    (stroke (width 1) (type default))
+  )
   (wire (pts (xy 101.6 130.81) (xy 115.57 130.81))
     (stroke (width 0) (type default))
@@
     (stroke (width 0) (type default))
   )
-  (wire (pts (xy 124.46 91.44) (xy 95.25 91.44))
+  (wire (pts (xy 124.46 91.44) (xy 116.84 91.44))
     (stroke (width 1) (type default))
   )
@@
     (effects (font (size 4 4) (thickness 0.8) bold (color 0 0 0 1)))
   )
+  (text "7 AMP fuse installed\nby power train" (at 95.25 43.18 0)
+    (effects (font (size 1.27 1.27)) (justify left bottom))
+  )
   (label "CAN_High" (at 104.14 134.62 0) (fields_autoplaced)

Commit message: ...
Parts:
- renumbered BT2 to BT4, D1 to D5, D1 to D7
Connections:
- net LV_pwr is gone; now on net LV_High: U?.2 (Ready_Power), U?.4 (Charge_Power)
Changed lines of the file:
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@@
     (effects (font (size 1.27 1.27)) (justify right))
   )
-  (hierarchical_label "LV_pwr" (shape input) (at 95.25 111.76 90) (fields_autoplaced)
-    (effects (font (size 1.27 1.27) (thickness 0.254) bold (color 255 0 0 1)) (justify left))
+  (hierarchical_label "LV_High" (shape input) (at 95.25 111.76 90) (fields_autoplaced)
+    (effects (font (size 1.27 1.27) (thickness 0.254) bold) (justify left))
   )
   (hierarchical_label "CAN_Bus_Out" (shape input) (at 99.06 111.76 90) (fields_autoplaced)
@@
   (symbol (lib_id "Diode:1N4001") (at 241.3 40.64 0) (unit 1)
     (in_bom yes) (on_board yes) (dnp no)
-    (property "Reference" "D1" (at 241.3 35.56 90)
+    (property "Reference" "D5" (at 241.3 35.56 90)
       (effects (font (size 1.27 1.27)))
     )
@@
   (symbol (lib_id "Device:Battery") (at 82.55 43.18 0) (mirror y) (unit 1)
     (in_bom yes) (on_board yes) (dnp no) (fields_autoplaced)
-    (property "Reference" "BT2" (at 86.36 41.3385 0)
+    (property "Reference" "BT4" (at 86.36 41.3385 0)
       (effects (font (size 1.27 1.27)) (justify right))
     )
@@
   (symbol (lib_id "Diode:1N4001") (at 241.3 105.41 0) (unit 1)
     (in_bom yes) (on_board yes) (dnp no)
-    (property "Reference" "D1" (at 241.3 100.33 90)
-      (effects (font (size 1.27 1.27)))
-    )
+    (property "Reference" "D7" (at 241.3 100.33 90)
+      (effects (font (size 1.27 1.27)))
+    )
