File: KiCad/NR24_Schematic/Car_TractiveSystem_v2.kicad_sch (KiCad schematic)
At the start: 11 parts, among them J1 M_con, J2 F_con, K2 Key Switch Relay, M1 Zero_7R_Motor, SW3 100V E-stop (Right), SW4 100V E-stop (Left), U1 Sevcon_Gen4_Size6, U2 Throttle

Commit message: Updates
Parts:
- added U7: Brake (AiM Pressure Sensor), symbol CamachosSymbols:Throttle
Connections:
- net IMD/AIR_In: now reaches SW3.1 (A)
- new net  LV power: U7.3 (Vb)
- new net Analog to TI Board: U7.1 (Analog_Signal)
- new net LV GND: U7.2 (GND)
Other:
- sheet AMS Battery renamed AMS & Battery
- note added: "CAN GND = LV GND"

Commit message: Root Update
Connections:
- net IMD/AIR_In renamed AMS & Battery/HV + Low A
Other:
- sheet AMS & Battery ports: added CAN_Bus_Out, HV + High A, HV + Low A, LV_pwr (chrg), LV_pwr (dchrg); removed HV +

Commit message: NOV1 Changes w Clarks
Parts:
- added SW7: TI power switch, symbol CamachosSymbols:SW_SPST
Connections:
- net B-: no longer K2.2
- net  LV power: no longer names the net of U7.3 (Vb)
- net Analog to TI Board: no longer names the net of U7.1 (Analog_Signal)
- net LV GND: no longer names the net of U7.2 (GND)
- new net: K2.2, SW7.2 (B)
- new net IMD/STDWN_CT_IN: SW7.1 (A)
Other:
- sheet AMS & Battery ports: added none; removed CAN_GND, CAN_High, CAN_Low
- sheet Dash ports: added +12V out; removed none
- sheet IMD ports: added STDWN_CT_IN, STDWN_CT_OUT; removed AIR_In, AIR_Out
- sheet Ti Board ports: added CAN; removed none

Commit message: More Additions
Parts:
- added LA6: TSAL, symbol Device:Lamp
Connections:
- net B-: now also LA6.1 (-)
- net Dash/Key_SW +: now also LA6.2 (+)
Other:
- note added: "Mounted to Frame"
Changed lines of the file:
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@@
     (rev "Print 1")
   )
+  (junction (at 67.31 134.62) (diameter 0) (color 0 0 0 0)
+  )
   (junction (at 241.3 204.47) (diameter 0) (color 0 0 0 0)
   )
@@
   (junction (at 186.69 222.25) (diameter 0) (color 0 0 0 0)
   )
+  (junction (at 64.77 139.7) (diameter 0) (color 0 0 0 0)
+  )
   (junction (at 124.46 210.82) (diameter 0) (color 0 0 0 0)
   )
@@
     (stroke (width 0) (type default))
   )
+  (bus_entry (at 123.19 100.33) (size 2.54 2.54)
+    (stroke (width 0.75) (type default) (color 0 132 132 1))
+  )
   (bus_entry (at 232.41 184.15) (size 2.54 -2.54)
     (stroke (width 0) (type default))
@@
     (stroke (width 0) (type default))
   )
+  (bus_entry (at 180.34 207.01) (size 2.54 -2.54)
+    (stroke (width 0) (type default))
+  )
+  (bus_entry (at 96.52 252.73) (size 2.54 2.54)
+    (stroke (width 0) (type default))
+  )
+  (bus_entry (at 105.41 184.15) (size -2.54 -2.54)
+    (stroke (width 0) (type default))
+  )
+  (bus_entry (at 182.88 242.57) (size -2.54 2.54)
+    (stroke (width 0) (type default))
+  )
+  (bus_entry (at 96.52 260.35) (size 2.54 2.54)
+    (stroke (width 0) (type default))
+  )
+  (bus_entry (at 96.52 255.27) (size 2.54 2.54)
+    (stroke (width 0) (type default))
+  )
   (bus_entry (at 13.97 100.33) (size 2.54 2.54)
-    (stroke (width 0) (type default))
-  )
-  (bus_entry (at 180.34 207.01) (size 2.54 -2.54)
-    (stroke (width 0) (type default))
-  )
-  (bus_entry (at 96.52 252.73) (size 2.54 2.54)
-    (stroke (width 0) (type default))
-  )
-  (bus_entry (at 105.41 184.15) (size -2.54 -2.54)
-    (stroke (width 0) (type default))
-  )
-  (bus_entry (at 182.88 242.57) (size -2.54 2.54)
-    (stroke (width 0) (type default))
-  )
-  (bus_entry (at 123.19 100.33) (size 2.54 2.54)
-    (stroke (width 0) (type default))
-  )
-  (bus_entry (at 96.52 260.35) (size 2.54 2.54)
-    (stroke (width 0) (type default))
-  )
-  (bus_entry (at 96.52 255.27) (size 2.54 2.54)
-    (stroke (width 0) (type default))
+    (stroke (width 0.75) (type default) (color 0 132 132 1))
+  )
+  (bus_entry (at 270.51 100.33) (size 2.54 2.54)
+    (stroke (width 0.75) (type default) (color 0 132 132 1))
   )
   (bus_entry (at 274.32 229.87) (size 2.54 2.54)
@@
     (stroke (width 0) (type default))
   )
-  (bus_entry (at 270.51 100.33) (size 2.54 2.54)
-    (stroke (width 0) (type default))
-  )
   (bus_entry (at 179.07 201.93) (size 2.54 -2.54)
     (stroke (width 0) (type default))
@@
   )
   (bus_entry (at 294.64 100.33) (size 2.54 2.54)
-    (stroke (width 0) (type default))
+    (stroke (width 0.75) (type default) (color 0 132 132 1))
   )
   (bus_entry (at 232.41 179.07) (size 2.54 -2.54)
@@
     (stroke (width 0) (type default))
   )
+  (wire (pts (xy 49.53 134.62) (xy 67.31 134.62))
+    (stroke (width 0) (type default))
+  )
   (wire (pts (xy 118.11 257.81) (xy 115.57 257.81))
     (stroke (width 0) (type default))
   )
+  (wire (pts (xy 67.31 134.62) (xy 67.31 139.7))
+    (stroke (width 0) (type default))
+  )
   (wire (pts (xy 170.18 212.09) (xy 170.18 255.27))
     (stroke (width 0.5) (type default))
@@
     (stroke (width 0) (type default))
   )
+  (wire (pts (xy 49.53 139.7) (xy 49.53 134.62))
+    (stroke (width 0) (type default))
+  )
   (polyline (pts (xy 166.37 208.28) (xy 177.8 208.28))
     (stroke (width 0.5) (type default))
@@
     (stroke (width 0) (type default))
   )
-  (wire (pts (xy 64.77 130.81) (xy 64.77 142.24))
+  (wire (pts (xy 64.77 130.81) (xy 64.77 139.7))
     (stroke (width 0) (type default))
   )
@@
     (stroke (width 0) (type default))
   )
+  (wire (pts (xy 59.69 139.7) (xy 64.77 139.7))
+    (stroke (width 0) (type default))
+  )
   (bus (pts (xy 274.32 214.63) (xy 274.32 227.33))
     (stroke (width 0) (type default))
   )
   (bus (pts (xy 50.8 170.18) (xy 50.8 215.9))
+    (stroke (width 0) (type default))
+  )
+  (wire (pts (xy 64.77 139.7) (xy 64.77 142.24))
     (stroke (width 0) (type default))
   )
@@
     (stroke (width 0) (type default))
   )
-  (wire (pts (xy 67.31 130.81) (xy 67.31 139.7))
+  (wire (pts (xy 67.31 130.81) (xy 67.31 134.62))
     (stroke (width 0) (type default))
   )
@@
   (bus (pts (xy 16.51 102.87) (xy 16.51 215.9))
     (stroke (width 0.75) (type default) (color 0 132 132 1))
+  )
+  (rectangle (start 60.96 143.51) (end 60.96 143.51)
+    (stroke (width 0) (type default))
+    (fill (type none))
+  )
+  (rectangle (start 46.99 133.35) (end 62.23 143.51)
+    (stroke (width 0.5) (type default) (color 194 0 194 1))
+    (fill (type none))
   )
   (text_box ""
@@
     (fill (type none))
     (effects (font (size 1.27 1.27)) (justify left top))
+  )
+  (text "Mounted to Frame" (at 45.72 146.05 0)
+    (effects (font (size 1.27 1.27)) (justify left bottom))
   )
   (text "Car Tractive System" (at 195.58 27.94 0)
@@
         )
       )
+    )
+  )
+  (symbol (lib_name "Lamp_4") (lib_id "Device:Lamp") (at 54.61 139.7 180) (unit 1)
+    (in_bom yes) (on_board yes) (dnp no)
+    (property "Reference" "LA6" (at 48.26 140.97 0)
+      (effects (font (size 1.27 1.27)) (justify right))
+    )
+    (property "Value" "TSAL" (at 52.07 135.89 0)
+      (effects (font (size 1.27 1.27)) (justify right))
+    )
+    (property "Footprint" "" (at 52.07 139.7 0)
+      (effects (font (size 1.27 1.27)) hide)
+    )
+    (property "Datasheet" "~" (at 52.07 139.7 0)
+      (effects (font (size 1.27 1.27)) hide)
+    )
+    (pin "1")
+    (pin "2")
+    (instances
+      (project "Car_TractiveSystem_v2"
+        (path "/588b5c14-1813-4e1d-9dbe-940839ecebe3"
+          (reference "LA6") (unit 1)
+        )
+        (path "/588b5c14-1813-4e1d-9dbe-940839ecebe3/62b4fa84-4530-4bff-bc03-eb6ea850cb52"
+          (reference "LA6") (unit 1)
+        )
+      )

Commit message: ams with IMD inside
Connections:
- net AMS & Battery/HV + High A: now also F1.2, U1. (M3)
- net Cont1 Supply (+): no longer names the net of U1.4 (Cont1_Supply_(+))
- removed net HV_Switch_Box/HV+: F1.2, U1. (M3)
- net Line Contactor (Cont1): no longer names the net of U1.3 (Line_Contactor_(Cont1))
Other:
- removed sheet HV_Switch_Box
Changed lines of the file:
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@@
-    (stroke (width 0) (type default))
-  )
-  (bus_entry (at 105.41 186.69) (size -2.54 -2.54)
     (stroke (width 0) (type default))
   )
@@
   )
   (bus_entry (at 96.52 252.73) (size 2.54 2.54)
-    (stroke (width 0) (type default))
-  )
-  (bus_entry (at 105.41 184.15) (size -2.54 -2.54)
     (stroke (width 0) (type default))
   )
@@
     (stroke (width 0.75) (type default) (color 0 132 132 1))
   )
-  (bus_entry (at 274.32 229.87) (size 2.54 2.54)
+  (bus_entry (at 313.69 240.03) (size -2.54 2.54)
     (stroke (width 0) (type default))
   )
@@
     (stroke (width 0) (type default))
   )
-  (bus_entry (at 181.61 181.61) (size -2.54 2.54)
-    (stroke (width 0) (type default))
-  )
   (bus_entry (at 179.07 201.93) (size 2.54 -2.54)
     (stroke (width 0) (type default))
@@
     (stroke (width 0) (type default))
   )
-  (bus_entry (at 274.32 227.33) (size 2.54 2.54)
+  (bus_entry (at 313.69 237.49) (size -2.54 2.54)
     (stroke (width 0) (type default))
   )
@@
     (stroke (width 0) (type default))
   )
-  (bus_entry (at 181.61 184.15) (size -2.54 2.54)
-    (stroke (width 0) (type default))
-  )
-  (bus_entry (at 274.32 232.41) (size 2.54 2.54)
+  (bus_entry (at 313.69 242.57) (size -2.54 2.54)
     (stroke (width 0) (type default))
   )
@@
     (stroke (width 0) (type default))
   )
-  (bus (pts (xy 274.32 227.33) (xy 274.32 229.87))
+  (bus (pts (xy 313.69 237.49) (xy 313.69 240.03))
     (stroke (width 0) (type default))
   )
@@
     (stroke (width 0) (type default))
   )
-  (wire (pts (xy 102.87 189.23) (xy 166.37 189.23))
-    (stroke (width 0.75) (type default))
-  )
   (polyline (pts (xy 173.99 215.9) (xy 173.99 259.08))
     (stroke (width 0.5) (type default))
@@
     (stroke (width 0) (type default))
   )
-  (bus (pts (xy 274.32 214.63) (xy 274.32 227.33))
-    (stroke (width 0) (type default))
-  )
   (bus (pts (xy 50.8 170.18) (xy 50.8 215.9))
     (stroke (width 0) (type default))
@@
     (stroke (width 0) (type default))
   )
-  (bus (pts (xy 313.69 214.63) (xy 274.32 214.63))
-    (stroke (width 0) (type default))
-  )
   (wire (pts (xy 143.51 135.89) (xy 143.51 144.78))
     (stroke (width 0) (type default))
@@
     (stroke (width 1) (type default) (color 0 132 132 1))
   )
-  (wire (pts (xy 276.86 232.41) (xy 279.4 232.41))
+  (wire (pts (xy 311.15 242.57) (xy 308.61 242.57))
     (stroke (width 0) (type default))
   )
@@
   )
   (wire (pts (xy 69.85 135.89) (xy 143.51 135.89))
-    (stroke (width 0) (type default))
-  )
-  (wire (pts (xy 181.61 184.15) (xy 186.69 184.15))
     (stroke (width 0) (type default))
   )
@@
     (stroke (width 0) (type default))
   )
-  (wire (pts (xy 279.4 229.87) (xy 276.86 229.87))
-    (stroke (width 0) (type default))
-  )
-  (bus (pts (xy 105.41 184.15) (xy 105.41 186.69))
+  (wire (pts (xy 308.61 240.03) (xy 311.15 240.03))
     (stroke (width 0) (type default))
   )
@@
     (stroke (width 0.5) (type default))
   )
-  (wire (pts (xy 55.88 189.23) (xy 81.28 189.23))
-    (stroke (width 0.75) (type default))
-  )
   (wire (pts (xy 116.84 176.53) (xy 116.84 163.83))
     (stroke (width 0.5) (type default))
@@
     (stroke (width 0) (type default))
   )
-  (bus (pts (xy 274.32 229.87) (xy 274.32 232.41))
+  (bus (pts (xy 313.69 240.03) (xy 313.69 242.57))
     (stroke (width 0) (type default))
   )
@@
     (stroke (width 0) (type default))
   )
-  (bus (pts (xy 105.41 184.15) (xy 179.07 184.15))
-    (stroke (width 0) (type default))
-  )
   (wire (pts (xy 60.96 207.01) (xy 71.12 207.01))
     (stroke (width 0) (type default))
   )
-  (wire (pts (xy 181.61 181.61) (xy 186.69 181.61))
-    (stroke (width 0) (type default))
-  )
   (bus (pts (xy 96.52 245.11) (xy 96.52 250.19))
     (stroke (width 0) (type default))
@@
     (stroke (width 0) (type default))
   )
-  (wire (pts (xy 276.86 234.95) (xy 279.4 234.95))
+  (wire (pts (xy 311.15 245.11) (xy 308.61 245.11))
     (stroke (width 0) (type default))
   )
@@
     (stroke (width 0) (type default))
   )
-  (bus (pts (xy 179.07 186.69) (xy 179.07 184.15))
-    (stroke (width 0) (type default))
-  )
   (wire (pts (xy 135.89 158.75) (xy 137.16 158.75))
     (stroke (width 0) (type default))
   )
-  (bus (pts (xy 313.69 148.59) (xy 313.69 214.63))
+  (bus (pts (xy 313.69 148.59) (xy 313.69 237.49))
     (stroke (width 0) (type default))
   )
@@
   )
   (wire (pts (xy 55.88 222.25) (xy 45.72 222.25))
+    (stroke (width 0.75) (type default))
+  )
+  (wire (pts (xy 55.88 189.23) (xy 166.37 189.23))
     (stroke (width 0.75) (type default))
   )
@@
     (effects (font (size 1.27 1.27)) (justify left bottom))
   )
-  (label "Cont1 Supply (+)" (at 181.61 184.15 180) (fields_autoplaced)
-    (effects (font (size 1.27 1.27)) (justify right bottom))
-  )
   (label "TI Board Inputs" (at 50.8 198.12 90) (fields_autoplaced)
     (effects (font (size 1.27 1.27)) (justify left bottom))
   )
-  (label "Line Contactor" (at 138.43 184.15 0) (fields_autoplaced)
-    (effects (font (size 1.27 1.27)) (justify left bottom))
-  )
-  (label "Line Contactor (Cont1)" (at 181.61 181.61 180) (fields_autoplaced)
-    (effects (font (size 1.27 1.27)) (justify right bottom))
-  )
   (label "LV Battery Ground" (at 124.46 208.28 90) (fields_autoplaced)
     (effects (font (size 1.27 1.27)) (justify left bottom))
@@
       (effects (font (size 1.27 1.27)) hide)
     )
-    (property "Value" "Throttle" (at 294.64 198.12 0)
-      (effects (font (size 1.27 1.27)) (justify left))
+    (property "Value" "Throttle" (at 297.18 199.39 0)
+      (effects (font (size 2 2)) (justify left))
     )
     (property "Footprint" "" (at 290.83 203.2 0)
@@
     )
   )
-  (symbol (lib_name "Throttle_1") (lib_id "CamachosSymbols:Throttle") (at 289.56 231.14 0) (unit 1)
-    (in_bom yes) (on_board yes) (dnp no)
-    (property "Reference" "U7" (at 304.8 227.33 0)
-      (effects (font (size 1.27 1.27)) hide)
-    )
-    (property "Value" "Brake (AiM Pressure Sensor)" (at 283.21 224.79 0)
-      (effects (font (size 1.27 1.27)) (justify left))
-    )
-    (property "Footprint" "" (at 289.56 231.14 0)
-      (effects (font (size 1.27 1.27)) hide)
-    )
-    (property "Datasheet" "" (at 289.56 231.14 0)
+  (symbol (lib_name "Throttle_1") (lib_id "CamachosSymbols:Throttle") (at 298.45 241.3 0) (mirror y) (unit 1)
+    (in_bom yes) (on_board yes) (dnp no)
+    (property "Reference" "U7" (at 283.21 237.49 0)
+      (effects (font (size 1.27 1.27)) hide)
+    )
+    (property "Value" "Brake (AiM Pressure Sensor)" (at 311.15 247.65 0)
+      (effects (font (size 1.27 1.27)) (justify left))
+    )
+    (property "Footprint" "" (at 298.45 241.3 0)
+      (effects (font (size 1.27 1.27)) hide)
+    )
+    (property "Datasheet" "" (at 298.45 241.3 0)
       (effects (font (size 1.27 1.27)) hide)
     )
@@
       )
     )
-  )
-  (sheet (at 81.28 179.07) (size 21.59 12.7) (fields_autoplaced)
-    (stroke (width 0.1524) (type solid))
-    (fill (color 0 0 0 0.0000))
-    (property "Sheetname" "HV_Switch_Box" (at 81.28 177.9934 0)
-      (effects (font (size 2 2)) (justify left bottom))
-    )
-    (property "Sheetfile" "HV_Switch_Box.kicad_sch" (at 81.28 192.3546 0)
-      (effects (font (size 1.27 1.27)) (justify left top))
-    )
-    (pin "HV -" input (at 81.28 189.23 180)
-      (effects (font (size 1.27 1.27)) (justify left))
-    )
-    (pin "HV+" input (at 102.87 189.23 0)
-      (effects (font (size 1.27 1.27)) (justify right))
-    )
-    (pin "Cont1" input (at 102.87 181.61 0)
-      (effects (font (size 1.27 1.27)) (justify right))
-    )
-    (pin "Cont1_Supply (+)" input (at 102.87 184.15 0)
-      (effects (font (size 1.27 1.27)) (justify right))
-    )
-    (instances
-      (project "Car_TractiveSystem_v2"
-        (path "/588b5c14-1813-4e1d-9dbe-940839ecebe3" (page "5"))
-      )
-    )
