File: KiCad/NR24_Schematic/IMD.kicad_sch (KiCad schematic)
At the start: 4 parts

Commit message: NOV1 Changes w Clarks
Connections:
- net AIR_In renamed STDWN_CT_IN
- net AIR_Out renamed STDWN_CT_OUT
Changed lines of the file:
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@@
     (effects (font (size 1.27 1.27)) (justify left))
   )
-  (hierarchical_label "AIR_In" (shape input) (at 162.56 77.47 180) (fields_autoplaced)
+  (hierarchical_label "STDWN_CT_IN" (shape input) (at 162.56 77.47 180) (fields_autoplaced)
     (effects (font (size 1.27 1.27)) (justify right))
   )
@@
     (effects (font (size 1.27 1.27)) (justify left))
   )
-  (hierarchical_label "AIR_Out" (shape input) (at 162.56 81.28 180) (fields_autoplaced)
+  (hierarchical_label "STDWN_CT_OUT" (shape input) (at 162.56 81.28 180) (fields_autoplaced)
     (effects (font (size 1.27 1.27)) (justify right))
   )
