File: KiCad/NR24_Schematic/IMD.kicad_sch (KiCad schematic)
At the start: 4 parts

Commit message: slight changes
Parts:
- renumbered D1 to D4
Changed lines of the file:
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@@
   (symbol (lib_id "Diode:1N4001") (at 194.31 81.28 270) (unit 1)
     (in_bom yes) (on_board yes) (dnp no)
-    (property "Reference" "D1" (at 199.39 81.28 90)
+    (property "Reference" "D4" (at 199.39 81.28 90)
       (effects (font (size 1.27 1.27)))
     )
