File: KiCad/NR24_Schematic/_autosave-Car_TractiveSystem_v2.kicad_sch (KiCad schematic)
At the start: 15 parts, among them J1 M_con, J2 F_con, K2 Key Switch Relay, M1 Zero_7R_Motor, SW3 100V E-stop (Right), SW4 100V E-stop (Left), SW7 TI power switch, SW8 GLVMS, U1 Sevcon_Gen4_Size6, U2 Throttle, U7 Brake (AiM Pressure Sensor)

Commit message: ..
Parts:
- 3A: value Fuse -> 3A Fuse
Other:
- moved on the sheet: SW8
