File: KiCad/NR24_Schematic/Dash.kicad_sch (KiCad schematic)
At the start: 11 parts, among them J9 AEM Dash, SW1 TI power switch, SW2 Shifter Switch, SW5 Key Switch, SW6 12V E-stop

Commit message: NOV1 Changes w Clarks
Connections:
- net 12V Power: no longer J9.1 (12V_Battery+), SW6.2 (B)
- net 12V+ to TI: now also J9.1 (12V_Battery+), SW6.2 (B)

Commit message: More Additions
Parts:
- SW1: value TI power switch -> GLVMS
Other:
- note added: "independent CAN watchdoggy device"
Changed lines of the file:
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@@
 (kicad_sch (version 20230121) (generator eeschema)
   (paper "A4")
+  (junction (at 166.37 123.19) (diameter 0) (color 0 0 0 0)
+  )
   (junction (at 236.22 142.24) (diameter 0) (color 0 0 0 0)
   )
@@
     (stroke (width 0) (type default))
   )
+  (bus_entry (at 218.44 76.2) (size 2.54 2.54)
+    (stroke (width 0) (type default))
+  )
   (bus_entry (at 49.53 59.69) (size -2.54 2.54)
     (stroke (width 0) (type default))
@@
     (stroke (width 0) (type default))
   )
+  (wire (pts (xy 156.21 96.52) (xy 148.59 96.52))
+    (stroke (width 0) (type default))
+  )
   (wire (pts (xy 127 101.6) (xy 140.97 101.6))
     (stroke (width 0) (type default))
   )
+  (bus (pts (xy 220.98 78.74) (xy 231.14 78.74))
+    (stroke (width 0.75) (type default) (color 0 132 132 1))
+  )
+  (wire (pts (xy 144.78 92.71) (xy 144.78 87.63))
+    (stroke (width 0) (type default))
+  )
   (wire (pts (xy 78.74 92.71) (xy 78.74 113.03))
     (stroke (width 0) (type default))
@@
     (stroke (width 0) (type default))
   )
+  (wire (pts (xy 148.59 96.52) (xy 148.59 92.71))
+    (stroke (width 0) (type default))
+  )
   (wire (pts (xy 138.43 123.19) (xy 138.43 151.13))
     (stroke (width 0) (type default))
   )
+  (wire (pts (xy 146.05 72.39) (xy 149.86 72.39))
+    (stroke (width 0) (type default))
+  )
+  (wire (pts (xy 203.2 69.85) (xy 203.2 68.58))
+    (stroke (width 0) (type default))
+  )
   (bus (pts (xy 77.47 62.23) (xy 102.87 62.23))
     (stroke (width 0) (type default))
@@
     (stroke (width 0) (type default))
   )
+  (wire (pts (xy 175.26 69.85) (xy 203.2 69.85))
+    (stroke (width 0) (type default))
+  )
   (wire (pts (xy 187.96 88.9) (xy 205.74 88.9))
     (stroke (width 0) (type default))
@@
     (stroke (width 0) (type default))
   )
+  (wire (pts (xy 175.26 66.04) (xy 175.26 69.85))
+    (stroke (width 0) (type default))
+  )
   (wire (pts (xy 74.93 64.77) (xy 74.93 82.55))
     (stroke (width 0) (type default))
@@
     (stroke (width 0) (type default))
   )
+  (wire (pts (xy 210.82 68.58) (xy 210.82 72.39))
+    (stroke (width 0) (type default))
+  )
   (wire (pts (xy 156.21 59.69) (xy 156.21 52.07))
     (stroke (width 0) (type default))
@@
   )
   (bus (pts (xy 110.49 62.23) (xy 113.03 62.23))
+    (stroke (width 0) (type default))
+  )
+  (wire (pts (xy 218.44 72.39) (xy 218.44 76.2))
+    (stroke (width 0) (type default))
+  )
+  (wire (pts (xy 149.86 72.39) (xy 149.86 66.04))
     (stroke (width 0) (type default))
   )
@@
     (stroke (width 0) (type default))
   )
+  (wire (pts (xy 149.86 66.04) (xy 175.26 66.04))
+    (stroke (width 0) (type default))
+  )
   (bus (pts (xy 179.07 62.23) (xy 231.14 62.23))
     (stroke (width 0) (type default))
@@
     (stroke (width 0) (type default))
   )
-  (wire (pts (xy 157.48 123.19) (xy 177.8 123.19))
+  (wire (pts (xy 157.48 123.19) (xy 166.37 123.19))
     (stroke (width 0) (type default))
   )
@@
     (stroke (width 0) (type default))
   )
+  (wire (pts (xy 148.59 92.71) (xy 144.78 92.71))
+    (stroke (width 0) (type default))
+  )
   (wire (pts (xy 138.43 113.03) (xy 205.74 113.03))
     (stroke (width 0) (type default))
   )
-  (bus (pts (xy 200.66 78.74) (xy 231.14 78.74))
+  (bus (pts (xy 200.66 78.74) (xy 220.98 78.74))
     (stroke (width 0.75) (type default) (color 0 132 132 1))
   )
@@
     (stroke (width 0) (type default))
   )
+  (wire (pts (xy 161.29 99.06) (xy 156.21 99.06))
+    (stroke (width 0) (type default))
+  )
   (bus (pts (xy 102.87 62.23) (xy 110.49 62.23))
     (stroke (width 0) (type default))
@@
     (stroke (width 0) (type default))
   )
+  (wire (pts (xy 166.37 104.14) (xy 166.37 123.19))
+    (stroke (width 0) (type default))
+  )
   (wire (pts (xy 165.1 52.07) (xy 167.64 52.07))
     (stroke (width 0) (type default))
@@
     (stroke (width 0) (type default))
   )
+  (wire (pts (xy 146.05 72.39) (xy 146.05 87.63))
+    (stroke (width 0) (type default))
+  )
   (bus (pts (xy 137.16 62.23) (xy 143.51 62.23))
     (stroke (width 0) (type default))
@@
     (stroke (width 0) (type default))
   )
+  (wire (pts (xy 203.2 68.58) (xy 210.82 68.58))
+    (stroke (width 0) (type default))
+  )
   (wire (pts (xy 181.61 52.07) (xy 181.61 59.69))
     (stroke (width 0) (type default))
@@
     (stroke (width 0) (type default))
   )
+  (wire (pts (xy 210.82 72.39) (xy 218.44 72.39))
+    (stroke (width 0) (type default))
+  )
+  (wire (pts (xy 156.21 99.06) (xy 156.21 96.52))
+    (stroke (width 0) (type default))
+  )
   (wire (pts (xy 242.57 142.24) (xy 242.57 102.87))
     (stroke (width 0) (type default))
@@
     (stroke (width 0) (type default))
   )
+  (wire (pts (xy 144.78 87.63) (xy 146.05 87.63))
+    (stroke (width 0) (type default))
+  )
   (wire (pts (xy 205.74 88.9) (xy 205.74 113.03))
     (stroke (width 0) (type default))
@@
     (stroke (width 0) (type default))
   )
+  (wire (pts (xy 166.37 123.19) (xy 177.8 123.19))
+    (stroke (width 0) (type default))
+  )
   (wire (pts (xy 152.4 52.07) (xy 156.21 52.07))
     (stroke (width 0) (type default))
@@
   (bus (pts (xy 43.18 62.23) (xy 46.99 62.23))
     (stroke (width 0) (type default))
+  )
+  (rectangle (start 161.29 97.79) (end 171.45 104.14)
+    (stroke (width 0) (type default) (color 72 0 0 1))
+    (fill (type color) (color 255 255 194 1))
+  )
+  (text "independent CAN \nwatchdoggy device\n" (at 160.02 102.87 0)
+    (effects (font (size 1 1)) (justify left bottom))
   )
   (text "|\\--/|\n| o_o |\n \\_ ^_/" (at 40.64 31.75 0)
@@
     )
   )
-  (global_label "CAN Bus" (shape input) (at 220.98 78.74 270) (fields_autoplaced)
+  (global_label "CAN Bus" (shape input) (at 227.33 78.74 270) (fields_autoplaced)
     (effects (font (size 1.27 1.27) (thickness 0.254) bold) (justify right))
-    (property "Intersheetrefs" "${INTERSHEET_REFS}" (at 220.98 90.305 90)
+    (property "Intersheetrefs" "${INTERSHEET_REFS}" (at 227.33 90.305 90)
       (effects (font (size 1.27 1.27)) (justify right) hide)
     )
@@
       (effects (font (size 1.27 1.27)))
     )
-    (property "Value" "TI power switch" (at 124.46 127 0)
-      (effects (font (size 1.27 1.27)))
-    )
+    (property "Value" "GLVMS" (at 124.46 127 0)
+      (effects (font (size 1.27 1.27)))
+    )

Commit message: Now it is pretty :)
Parts:
- removed LA4: Fault Light, symbol Device:Lamp
- removed SW1: GLVMS, symbol CamachosSymbols:SW_SPST
- added LA2: AMS Fault Batt L, symbol Device:Lamp
- added LA2: AMS Fault Batt H, symbol Device:Lamp
Connections:
- net 12V+ to TI is gone; now on net 12V Power: J9.1 (12V_Battery+), LA1.2 (+), SW6.2 (B)
- net 12V GND to TI renamed Earth
- net Dash Error + renamed 12V High
- net 12V High: now also LA2.2 (+), LA2.2 (+)
- net Dash Error -: no longer names the net of LA2.1 (-)
- net F_Light(+): no longer names the net of LA2.2 (+)
- net F_Light(-): no longer names the net of LA2.1 (-)
- net N_Light(+): no longer names the net of LA5.1 (-)
- net N_Light(-): no longer names the net of LA5.2 (+)
- net Rocker_1 renamed Rocker 1
- net Rocker_2 renamed Rocker 2
- net Rocker_3 renamed Rocker 3
Other:
- note removed: "independent CAN watchdoggy device"
- moved on the sheet: LA1, LA2, LA5, SW2, SW5, SW6

Commit message: slight changes
Other:
- note added: "DASH"
Changed lines of the file:
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@@
     (stroke (width 0) (type default))
   )
-  (text "|\\--/|\n| o_o |\n \\_ ^_/" (at 74.93 29.21 0)
+  (text "|\\--/|\n| o_o |\n \\_ ^_/" (at 12.7 27.94 0)
     (effects (font (size 3 3)) (justify left bottom))
   )
+  (text "DASH" (at 82.55 41.91 0)
+    (effects (font (size 4 4) (thickness 0.8) bold) (justify left bottom))
+  )
   (label "Dash +12V" (at 184.15 119.38 0) (fields_autoplaced)
