File: KiCad/NR24_Schematic/Battery_High.kicad_sch (KiCad schematic)
At the start: 9 parts

Commit message: Now it is pretty :)
Connections:
- net Dash_Error + renamed Dash_Error_AMS +
- net Dash_Error_AMS +: no longer RL3.2
- net Dash_Error - renamed Dash_Error_AMS -
- net Dash_Error_AMS -: no longer RL3.3
- new net Dash_Error_IMD +: RL3.2
- new net Dash_Error_IMD -: RL3.3
Other:
- moved on the sheet: BT4, D5, RL3
